File: Placa/SE/proyecto.kicad_pcb (KiCad board)
At the start: 2 copper layers, 12 parts, among them J1 Conn_01x02, J2 Conn_01x03, J3 Conn_01x05, J4 Conn_01x08, U1 LM7805_TO220, U2 PIC16F886-IP, Y1 Crystal

Commit message: added lamp project
Parts:
- moved C1 3.56 mm to (135.9, 78.7)
- moved C2 3.56 mm to (135.9, 85.1)
- moved J1 3.56 mm to (122.0, 85.1)
- moved U1 3.56 mm to (130.8, 80.0)
Routing:
- net GND: track 161.5 -> 170.0 mm
- net +5V: track 88.5 -> 87.8 mm
- net Net-(J3-Pad1): track 19.7 -> 20.3 mm
Other:
- net class Default removed
- net class Signal removed
